File: eagle_NAHS-SignalBrick/v1.0_r1.brd (EAGLE design)
At the start: 45.5 x 70.3 mm, 42 parts, among them IC1 ESP12F, IC2 ATTINY212-SSNR, IC3 TP4056, IC4 DW01A, J1 10118194-0001LF, J2 Brick-Interface, Q1 8205A

Commit message: renamed components, finished for production
Parts:
- removed C6, C7: 10µF, rcl:C0805
- added C1: 100nF, rcl:C0805
- added C3: 1µF, rcl:C0805
- C2: value 100nF -> 1µF
- C4, C5: value 1µF -> 10µF
- R10, R11: value 10k -> 3.9k
- R13: value 590k -> 10k
- R14: value 2.7M -> 10k
- R15: value 510 -> 10k; device rcl:R0603 -> rcl:R0805
- R16: value 510 -> 590k; device rcl:R0603 -> rcl:R0805
- R17: value 510 -> 2.7M; device rcl:R0603 -> rcl:R0805
- R3, R4, R5: value 1k -> 510; device rcl:R0805 -> rcl:R0603
- R6: value 1.74k -> 1k
- R7, R8: value 3.9k -> 1k
- R9: value 10k -> 1.74k
- moved R9 52.3 mm to (25.4, 64.8)
- moved R12 45.0 mm to (20.3, 12.7), turned to 0 degrees
- moved R7 34.8 mm to (23.2, 52.5), turned to 90 degrees
- moved R5 26.7 mm to (30.5, 34.8), turned to 270 degrees
- moved R14 23.2 mm to (20.3, 22.9), turned to 0 degrees
- moved R13 22.9 mm to (20.3, 20.3), turned to 0 degrees
- moved R15 22.2 mm to (30.1, 56.6), turned to 90 degrees
- moved R6 20.8 mm to (27.7, 44.1), turned to 270 degrees
- moved C4 20.5 mm to (20.3, 52.1), turned to 270 degrees
- moved R4 18.3 mm to (28.2, 34.8), turned to 270 degrees
- moved C2 17.0 mm to (39.4, 44.5)
- moved C5 11.7 mm to (20.3, 44.5)
- moved R3 9.44 mm to (25.9, 34.8)
- moved R11 7.62 mm to (20.3, 15.2)
- moved R17 7.56 mm to (35.4, 40.5), turned to 180 degrees
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Connections:
- net +3V3: now also C3.1, R11.1, R12.1, R13.1; no longer C5.1, R7.1, R8.1, R9.1
- net A0: now also R16.1, R17.2; no longer R13.1, R14.2
- net BAT+: now also C5.1; no longer C7.1
- net BAT-: now also R6.1; no longer R3.1
- net BOOT1: now also R13.2; no longer R10.2
- net BOOT2: now also R14.2; no longer R11.2
- net CD: now also R15.2; no longer R12.2
- net CHRG: now also R7.2; no longer R4.2
- net EN: now also R12.2; no longer R9.2
- net GND: now also C2.2, C3.2, R14.1, R16.2; no longer C4.2, C5.2, R11.1, R13.2
- net IN-: now also C1.2, C4.2, C5.2, R9.1; no longer C2.2, C6.2, C7.2, R6.1
- net N$1: now also C4.1, R15.1; no longer C6.1, R12.1
- net N$2: now also R9.2; no longer R6.2
- net N$3: now also R6.2; no longer R3.2
- net N$4: now also C1.1; no longer C2.1
- net N$5: now also R3.2; no longer R15.2
- net N$6: now also R4.2; no longer R16.2
- net N$7: now also R7.1; no longer R4.1
- net N$9: now also R5.2; no longer R17.2
- net RST: now also R8.2; no longer R5.2
- net SCL: now also R11.2; no longer R8.2
- net SDA: now also R10.2; no longer R7.2
- net SEL+: now also C2.1, R17.1; no longer C4.1, R14.1
- net SIG1: now also R3.1; no longer R15.1
- net SIG2: now also R4.1; no longer R16.1
- net SIG3: now also R5.1; no longer R17.1
- net WAKE: now also R8.1; no longer R5.1
