File: eagle_NAHS-SignalBrick/v1.0_r2.brd (EAGLE design)
At the start: 45.5 x 70.3 mm, 42 parts, among them IC1 ESP12S, IC2 ATTINY212-SSNR, IC3 TP4056, IC4 DW01A, J1 10118194-0001LF, J2 NAHS-BRICK-INTERFACE-V2_B-SIDE, Q1 8205A

Commit message: Boardlayout for v1.0 R2
Parts:
- added FD1, FD2, FD3: (no value), no_reichelt:FIDUCIAL
- moved R 8.13 mm to (42.3, 25.5)
Routing:
- net GND: track 94.3 -> 168.4 mm
- net N$9: track 0.00 -> 9.03 mm
- net N$5: track 0.00 -> 4.96 mm
- net N$6: track 0.00 -> 3.93 mm
- net UPDI: track 37.4 -> 38.4 mm
- net IN-: track 123.9 -> 123.1 mm
- net +3V3: track 125.9 -> 126.6 mm
- added copper zone on layer 1, net GND
Other:
- board text added: "Brick-Interface-V2"

Commit message: Boardlayout v1.0 R2 - Send to JLCPCB
Parts:
- R3, R4, R5: value 510 -> 330
Changed lines of the file:
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@@
 <attribute name="VALUE" x="37.5666" y="31.0896" size="1.27" layer="27" ratio="10" rot="R270"/>
 </element>
-<element name="R3" library="rcl" library_urn="urn:adsk.eagle:library:334" package="R0603" package3d_urn="urn:adsk.eagle:package:23555/3" value="510" x="26.543" y="39.497" smashed="yes" rot="R270">
+<element name="R3" library="rcl" library_urn="urn:adsk.eagle:library:334" package="R0603" package3d_urn="urn:adsk.eagle:package:23555/3" value="330" x="26.543" y="39.497" smashed="yes" rot="R270">
 <attribute name="POPULARITY" value="70" x="26.543" y="39.497" size="1.778" layer="27" rot="R270" display="off"/>
 <attribute name="SPICEPREFIX" value="R" x="26.543" y="39.497" size="1.778" layer="27" rot="R270" display="off"/>
 </element>
-<element name="R4" library="rcl" library_urn="urn:adsk.eagle:library:334" package="R0603" package3d_urn="urn:adsk.eagle:package:23555/3" value="510" x="29.083" y="39.497" smashed="yes" rot="R270">
+<element name="R4" library="rcl" library_urn="urn:adsk.eagle:library:334" package="R0603" package3d_urn="urn:adsk.eagle:package:23555/3" value="330" x="29.083" y="39.497" smashed="yes" rot="R270">
 <attribute name="POPULARITY" value="70" x="29.083" y="39.497" size="1.778" layer="27" rot="R270" display="off"/>
 <attribute name="SPICEPREFIX" value="R" x="29.083" y="39.497" size="1.778" layer="27" rot="R270" display="off"/>
 </element>
-<element name="R5" library="rcl" library_urn="urn:adsk.eagle:library:334" package="R0603" package3d_urn="urn:adsk.eagle:package:23555/3" value="510" x="31.623" y="39.497" smashed="yes" rot="R270">
+<element name="R5" library="rcl" library_urn="urn:adsk.eagle:library:334" package="R0603" package3d_urn="urn:adsk.eagle:package:23555/3" value="330" x="31.623" y="39.497" smashed="yes" rot="R270">
 <attribute name="POPULARITY" value="70" x="31.623" y="39.497" size="1.778" layer="27" rot="R270" display="off"/>
 <attribute name="SPICEPREFIX" value="R" x="31.623" y="39.497" size="1.778" layer="27" rot="R270" display="off"/>
