File: eagle_NAHS-SignalBrick/v1.0_r3.brd (EAGLE design)
At the start: 45.5 x 70.3 mm, 49 parts, among them IC1 ESP12S, IC2 ATTINY212-SSNR, IC3 TP4056, IC4 DW01A, J1 10118194-0001LF, J2 BRICK-INTERF-V3_B-SIDE, Q1 8205A

Commit message: Board v1.0 R3 WIP
Parts:
- added SJ4: DisableCharging, no_pinhd:SOLDERJUMPER
Connections:
- net CD: now also SJ4.2
- net IN-: now also SJ4.1
Routing:
- net IN-: track 123.3 -> 128.3 mm
- net CD: track 56.8 -> 61.7 mm, vias 0 -> 1
Other:
- board text added: "Disable Charging"
Changed lines of the file:
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@@
 <wire x1="29.21" y1="45.085" x2="26.035" y2="41.91" width="0.254" layer="52"/>
 <wire x1="38.735" y1="41.91" x2="35.56" y2="45.085" width="0.254" layer="52"/>
+<text x="25.4" y="65.405" size="1.27" layer="52" font="vector" ratio="10" rot="MR90" align="top-center">Disable
+Charging</text>
 </plain>
 <attributes>
@@
 <attribute name="VALUE" x="36.83" y="39.37" size="1.016" layer="28" font="vector" ratio="10" rot="MR0" align="bottom-center"/>
 </element>
+<element name="SJ4" library="no_pinhd" package="SOLDERJUMPER" value="DisableCharging" x="26.67" y="65.405" smashed="yes" rot="MR90">
+<attribute name="NAME" x="26.67" y="64.135" size="1.016" layer="26" font="vector" ratio="10" rot="MR90" align="center-right"/>
+</element>
 </elements>
 <signals>
@@
 <via x="34.26" y="64.74" extent="1-16" drill="0.35"/>
 <wire x1="34.26" y1="64.74" x2="32.5328" y2="64.74" width="0.8128" layer="16"/>
-<wire x1="32.5328" y1="64.74" x2="26.6192" y2="58.8264" width="0.8128" layer="16"/>
+<wire x1="32.5328" y1="64.74" x2="30.8864" y2="63.0936" width="0.8128" layer="16"/>
+<wire x1="30.8864" y1="63.0936" x2="26.6192" y2="58.8264" width="0.8128" layer="16"/>
 <wire x1="21.205" y1="48.585" x2="21.205" y2="48.26" width="0.254" layer="1"/>
 <wire x1="21.205" y1="47.935" x2="21.205" y2="48.26" width="0.254" layer="1"/>
@@
 <wire x1="11.04" y1="58.804" x2="13.081" y2="56.763" width="0.6096" layer="16"/>
 <wire x1="13.081" y1="56.763" x2="13.081" y2="51.689" width="0.6096" layer="16"/>
+<contactref element="SJ4" pad="1"/>
+<wire x1="26.67" y1="64.9732" x2="29.0068" y2="64.9732" width="0.254" layer="16"/>
+<wire x1="29.0068" y1="64.9732" x2="30.8864" y2="63.0936" width="0.254" layer="16"/>
+<wire x1="5.96" y1="58.804" x2="8.5" y2="66.424" width="0" layer="19" extent="1-1"/>
+<wire x1="11.04" y1="58.804" x2="5.96" y2="58.804" width="0" layer="19" extent="1-1"/>
 </signal>
 <signal name="N$2">
@@
 <wire x1="12.856" y1="36.674" x2="11.7674" y2="37.7626" width="0.254" layer="1"/>
 <wire x1="11.7674" y1="51.8133875" x2="21.7932" y2="61.8391875" width="0.254" layer="1"/>
+<contactref element="SJ4" pad="2"/>
+<wire x1="29.464" y1="64.704" x2="29.464" y2="66.5489" width="0.254" layer="1"/>
+<via x="29.464" y="66.5489" extent="1-16" drill="0.35"/>
+<wire x1="26.67" y1="65.8368" x2="28.7519" y2="65.8368" width="0.254" layer="16"/>
+<wire x1="28.7519" y1="65.8368" x2="29.464" y2="66.5489" width="0.254" layer="16"/>
 </signal>
 <signal name="SIG0">

Commit message: Board v1.0 R3 WIP
Parts:
- LED2: value (none) -> S0
- LED3: value (none) -> S1
- LED4: value (none) -> S2
- moved R8 2.54 mm to (20.3, 17.8)
- moved R9 2.54 mm to (20.3, 15.2)
- moved R5 2.54 mm to (20.3, 10.2)
- moved R10 2.54 mm to (20.3, 12.7)
Routing:
- net +3V3: track 130.2 -> 126.4 mm
- net SDA: track 54.6 -> 56.8 mm
- net SCL: track 58.0 -> 59.8 mm
- net RST: track 33.7 -> 35.3 mm
- net EN: track 21.6 -> 22.1 mm
Other:
- board text added: "3V3"
- board text added: "GND"
- board text added: "IN+"
- board text added: "IN-"
- board text added: "PROG"
- board text added: "RXD"
- board text added: "SETUP"
- board text added: "TXD"
- board text added: "UPDI"
- board text removed: "P"
- board text removed: "S"
- board text removed: "S0"
- board text removed: "S1"
- board text removed: "S2"
- board text removed: "U"

Commit message: Board v1.0 R3 done
Parts:
- R10, R11: value 10k -> 3.9k
- R14: value 590k -> 10k
- R15: value 2.7M -> 10k
- R16: value 330 -> 590k; device rcl:R0603 -> rcl:R0805
- R17: value 330 -> 2.7M; device rcl:R0603 -> rcl:R0805
- R3, R4, R5: value 1k -> 330; device rcl:R0805 -> rcl:R0603
- R6: value 1.74k -> 1k
- R7: value 330 -> 1k; device rcl:R0603 -> rcl:R0805
- R8: value 3.9k -> 1k
- R9: value 3.9k -> 1.74k
- SJ1: value S0 -> DisableCharging
- SJ2: value S1 -> S0
- SJ3: value S2 -> S1
- SJ4: value DisableCharging -> S2
- moved R13 51.9 mm to (20.3, 12.7), turned to 0 degrees
- moved R9 49.8 mm to (25.4, 64.8)
- moved R12 41.9 mm to (29.5, 63.8), turned to 90 degrees
- moved R14 33.4 mm to (20.3, 20.3), turned to 0 degrees
- moved R15 33.4 mm to (20.3, 22.9), turned to 0 degrees
- moved R5 32.5 mm to (36.8, 38.1), turned to 270 degrees
- moved SJ4 29.1 mm to (36.8, 38.1)
- moved SJ1 27.3 mm to (26.7, 65.4)
- moved R4 17.0 mm to (32.4, 38.1), turned to 270 degrees
- moved R17 12.7 mm to (38.7, 50.7), turned to 180 degrees
- moved R16 12.7 mm to (34.2, 50.7), turned to 180 degrees
- moved R6 12.5 mm to (23.2, 52.5), turned to 90 degrees
- moved R8 7.62 mm to (20.3, 10.2), turned to 180 degrees
- moved R3 5.97 mm to (27.9, 38.1)
- moved R7 5.97 mm to (27.7, 44.1)
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Connections:
- net +3V3: now also R13.1, R14.1; no longer R8.1, R9.1
- net A0: now also R16.1, R17.2; no longer R14.1, R15.2
- net BAT-: now also R7.1; no longer R3.1
- net BOOT1: now also R14.2; no longer R11.2
- net BOOT2: now also R15.2; no longer R12.2
- net CD: now also R12.2, SJ1.2; no longer R13.2, SJ4.2
- net CHRG: now also R6.2; no longer R4.2
- net EN: now also R13.2; no longer R10.2
- net GND: now also R15.1, R16.2; no longer R12.1, R14.2
- net IN-: now also R9.1, SJ1.1; no longer R6.1, SJ4.1
- net N$1: now also R12.1; no longer R13.1
- net N$2: now also R9.2; no longer R6.2
- net N$3: now also R7.2; no longer R3.2
- net N$5: now also R3.2, SJ2.1; no longer R7.2, SJ1.1
- net N$6: now also R4.2, SJ3.1; no longer R16.2, SJ2.1
- net N$7: now also R6.1; no longer R4.1
- net N$9: now also R5.2, SJ4.1; no longer R17.2, SJ3.1
- net RST: now also R8.2; no longer R5.2
- net SCL: now also R10.2; no longer R9.2
- net SDA: now also R11.2; no longer R8.2
- net SEL+: now also R17.1; no longer R15.1
- net SIG0: now also R3.1, SJ2.2; no longer R7.1, SJ1.2
- net SIG1: now also R4.1, SJ3.2; no longer R16.1, SJ2.2
- net SIG2: now also R5.1, SJ4.2; no longer R17.1, SJ3.2
- net WAKE: now also R8.1; no longer R5.1
Other:
- board text added: "NAHS-SignalBrick"
- board text added: "v1.0 R3"
- board text removed: "NAHS-RHTBrick"
- board text removed: "v1.0 R2"
