File: eagle_NAHS-SignalBrick/v1.0_r3.sch (EAGLE design)
At the start: 45 parts, among them IC1 ESP12S, IC2 ATTINY212-SSNR, IC3 TP4056, IC4 DW01A, J1 10118194-0001LF, J2 BRICK-INTERF-V3_B-SIDE, Q1 8205A

Commit message: Board v1.0 R3 WIP
Parts:
- added SJ4: DisableCharging, no_pinhd:SOLDERJUMPER
Connections:
- net CD: now also SJ4.2
- net IN-: now also SJ4.1
Other:
- moved on the sheet: C5, IC3, LED1, R1, R13, R4, R6

Commit message: Board v1.0 R3 WIP
Parts:
- LED2: value (none) -> S0
- LED3: value (none) -> S1
- LED4: value (none) -> S2
Changed lines of the file:
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@@
 <part name="J2" library="no_brick_interface" deviceset="BRICK-INTERF-V3" device="_B-SIDE"/>
 <part name="+3V5" library="supply1" library_urn="urn:adsk.eagle:library:371" deviceset="+3V3" device=""/>
-<part name="LED2" library="led" library_urn="urn:adsk.eagle:library:259" deviceset="LED" device="5MM" package3d_urn="urn:adsk.eagle:package:15799/2"/>
-<part name="LED3" library="led" library_urn="urn:adsk.eagle:library:259" deviceset="LED" device="5MM" package3d_urn="urn:adsk.eagle:package:15799/2"/>
-<part name="LED4" library="led" library_urn="urn:adsk.eagle:library:259" deviceset="LED" device="5MM" package3d_urn="urn:adsk.eagle:package:15799/2"/>
+<part name="LED2" library="led" library_urn="urn:adsk.eagle:library:259" deviceset="LED" device="5MM" package3d_urn="urn:adsk.eagle:package:15799/2" value="S0"/>
+<part name="LED3" library="led" library_urn="urn:adsk.eagle:library:259" deviceset="LED" device="5MM" package3d_urn="urn:adsk.eagle:package:15799/2" value="S1"/>
+<part name="LED4" library="led" library_urn="urn:adsk.eagle:library:259" deviceset="LED" device="5MM" package3d_urn="urn:adsk.eagle:package:15799/2" value="S2"/>
 <part name="R7" library="rcl" library_urn="urn:adsk.eagle:library:334" deviceset="R-EU_" device="R0603" package3d_urn="urn:adsk.eagle:package:23555/3" value="330"/>
 <part name="R16" library="rcl" library_urn="urn:adsk.eagle:library:334" deviceset="R-EU_" device="R0603" package3d_urn="urn:adsk.eagle:package:23555/3" value="330"/>

Commit message: Board v1.0 R3 done
Parts:
- R10, R11: value 10k -> 3.9k
- R14: value 590k -> 10k
- R15: value 2.7M -> 10k
- R16: value 330 -> 590k; device rcl:R-EU_R0603 -> rcl:R-EU_R0805
- R17: value 330 -> 2.7M; device rcl:R-EU_R0603 -> rcl:R-EU_R0805
- R3, R4, R5: value 1k -> 330; device rcl:R-EU_R0805 -> rcl:R-EU_R0603
- R6: value 1.74k -> 1k
- R7: value 330 -> 1k; device rcl:R-EU_R0603 -> rcl:R-EU_R0805
- R8: value 3.9k -> 1k
- R9: value 3.9k -> 1.74k
- SJ1: value S0 -> DisableCharging
- SJ2: value S1 -> S0
- SJ3: value S2 -> S1
- SJ4: value DisableCharging -> S2
Connections:
- net +3V3: now also R13.1, R14.1; no longer R8.1, R9.1
- net A0: now also R16.1, R17.2; no longer R14.1, R15.2
- net BAT-: now also R7.1; no longer R3.1
- net BOOT1: now also R14.2; no longer R11.2
- net BOOT2: now also R15.2; no longer R12.2
- net CD: now also R12.2, SJ1.2; no longer R13.2, SJ4.2
- net CHRG: now also R6.2; no longer R4.2
- net EN: now also R13.2; no longer R10.2
- net GND: now also R15.1, R16.2; no longer R12.1, R14.2
- net IN-: now also R9.1, SJ1.1; no longer R6.1, SJ4.1
- net N$1: now also R12.1; no longer R13.1
- net N$2: now also R9.2; no longer R6.2
- net N$3: now also R7.2; no longer R3.2
- net N$5: now also R3.2, SJ2.1; no longer R7.2, SJ1.1
- net N$6: now also R4.2, SJ3.1; no longer R16.2, SJ2.1
- net N$7: now also R6.1; no longer R4.1
- net N$9: now also R5.2, SJ4.1; no longer R17.2, SJ3.1
- net RST: now also R8.2; no longer R5.2
- net SCL: now also R10.2; no longer R9.2
- net SDA: now also R11.2; no longer R8.2
- net SEL+: now also R17.1; no longer R15.1
- net SIG0: now also R3.1, SJ2.2; no longer R7.1, SJ1.2
- net SIG1: now also R4.1, SJ3.2; no longer R16.1, SJ2.2
- net SIG2: now also R5.1, SJ4.2; no longer R17.1, SJ3.2
- net WAKE: now also R8.1; no longer R5.1
Other:
- moved on the sheet: BT1, C5, IC1, IC2, IC3, JP2_1, JP2_2, JP2_3, LED1, LED2, LED3, LED4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
